Commit message: 整体逻辑仿真通过,等待现实调参

File: src/conqu_vision/model/base.urdf (robot description, URDF)
Before this commit: robot rc_baseplate, 8 links, 7 joints
Links:
- removed link base_footprint
- removed link laser2_link
- removed link wheel_lb
- removed link wheel_lf
- removed link wheel_rb
- removed link wheel_rf
Joints:
- removed joint base_joint
- removed joint base_to_laser2
- removed joint base_to_wheel_lb
- removed joint base_to_wheel_lf
- removed joint base_to_wheel_rb
- removed joint base_to_wheel_rf
- joint base_to_laser1: origin xyz=0 0.279725 0 rpy=3.14159 0 1.5708 -> xyz=0 -0.32 0.15 rpy=3.14159 0 1.5708
